Commit message: Added gazebo reference for colour

File: src/articubot_one/description/robot_core.xacro (robot description, xacro)
@@ -51,4 +51,7 @@
         </xacro:inertial_box>
     </link>
+    <gazebo reference="chassis">
+        <material>Gazebo/White</material>
+    </gazebo>
     <!-- LEFT WHEEL LINK-->
 <!--Wheel will be connect to either base_link or Chassis using a continuous joint type-->
@@ -77,4 +80,7 @@
         </xacro:inertial_cylinder>
     </link>
+    <gazebo reference="left_wheel">
+        <material>Gazebo/Black</material>
+    </gazebo>
     <!-- RIGHT WHEEL LINK-->
 <!--Wheel will be connect to either base_link or Chassis using a continuous joint type-->
@@ -103,4 +109,7 @@
         </xacro:inertial_cylinder>
     </link>
+    <gazebo reference="right_wheel">
+        <material>Gazebo/Black</material>
+    </gazebo>
     <!-- CASTER WHEEL LINK -->
 <!--the default position of child link is the origin of parent so we need to move caster to the front (almost 0.24m in +x)-->
@@ -126,3 +135,6 @@
         </xacro:inertial_sphere>
     </link>
+    <gazebo reference="caster_wheel">
+        <material>Gazebo/Blue</material>
+    </gazebo>
 </robot>
