Commit message: LIDAR
Added lidar plugin and lidar.xacro file to add lidar fuctionality to robot

File: src/articubot_one/description/robot.urdf.xacro (robot description, xacro)
@@ -4,3 +4,4 @@
 	<xacro:include filename="robot_core.xacro"/>
 	<xacro:include filename="gazebo_control.xacro"/>
+	<xacro:include filename="lidar.xacro"/>
 </robot>

File: src/articubot_one/description/robot_core.xacro (robot description, xacro)
@@ -18,8 +18,10 @@
         <color rgba="0 0 0 1"/>
     </material>
+    <material name="red">
+        <color rgba="1 0 0 1"/>
+    </material>
     <!-- BASE LINK -->
 <!--Creating first link the ros standard for first link is "base_link"-->
-    <link name="base_link">
-    </link>
+    <link name="base_link"></link>
     <!-- CHASSIS LINK -->
 <!--Chassis is box which is 300mm 300mm 150mm urdf uses measurements in meters-->
@@ -31,5 +33,5 @@
     </joint>
 <!--Creating the chassis link which we joined to the base_link above using a fixed joint-->
-<!--By default the chassis link will bw centered around the chassis origin so we need to move the visuals of box
+<!--By default the chassis link will be centered around the chassis origin so we need to move the visuals of box
 we need to move it forward half its length(x) and up by half its height(z)-->
     <link name="chassis">
